File: BondTest72.kicad_pcb (KiCad board)
At the start: 4 copper layers, 80 x 100 mm, 79 parts, among them J1 Conn_01x07, J3 Conn_2Rows-41Pins_MountingPin, J4 Conn_2Rows-41Pins_MountingPin, SW1 SW_Push, SW2 K8-5851S-N1, SW3 K8-5851S-N1, U1 TPS7A0533PDBV, U2 CH446X, U3 CH446X, U4 CH446X

Commit message: - r2 update. Notes in README.md
Parts:
- removed C47: 100n, Capacitor_SMD:C_0201_0603Metric
- removed D3: SK6812, LED_SMD:LED_SK6812_PLCC4_5.0x5.0mm_P3.2mm
- removed JP3: SolderJumper_2_Open, Jumper:SolderJumper-2_P1.3mm_Open_TrianglePad1.0x1.5mm
- removed R10, R9: 1M, Resistor_SMD:R_0201_0603Metric
- removed SW3: K8-5851S-N1, lib:K8-5851S-N1
- removed kibuzzard-6A01FA95 (x2): G***, kibuzzard-6A01FA95
- removed kibuzzard-6A01FAD6: G***, kibuzzard-6A01FAD6
- removed kibuzzard-6A01FB6B: G***, kibuzzard-6A01FB6B
- removed kibuzzard-6A02741A: G***, kibuzzard-6A02741A
- removed kibuzzard-6A029CC3: G***, kibuzzard-6A029CC3
- removed kibuzzard-6A029D26: G***, kibuzzard-6A029D26
- removed kibuzzard-6A02B01A: G***, kibuzzard-6A02B01A
- removed kibuzzard-6A02B023: G***, kibuzzard-6A02B023
- removed kibuzzard-6A02B030: G***, kibuzzard-6A02B030
- removed kibuzzard-6A02B04E: G***, kibuzzard-6A02B04E
- removed kibuzzard-6A02B0B1: G***, kibuzzard-6A02B0B1
- added C23: 100n, Capacitor_SMD:C_0201_0603Metric, F.Cu at (83.2, 135.5)
- added C24: 100n, Capacitor_SMD:C_0201_0603Metric, F.Cu at (68.2, 135.5)
- added C25: 100n, Capacitor_SMD:C_0201_0603Metric, F.Cu at (53.2, 135.5)
- added C50: 120pF, Capacitor_SMD:C_0201_0603Metric, F.Cu at (50.2, 106.3)
- added R14: 10k, Resistor_SMD:R_0201_0603Metric, F.Cu at (32.2, 106.0)
- added R15: 100k, Resistor_SMD:R_0201_0603Metric, F.Cu at (75.2, 80.5)
- added kibuzzard-6AAFDF39: G***, kibuzzard-6AAFDF39, F.Cu at (103.0, 129.5)
- added kibuzzard-6AAFDFCA: G***, kibuzzard-6AAFDFCA, F.Cu at (103.0, 136.5)
- added kibuzzard-6AAFFF26: G***, kibuzzard-6AAFFF26, F.Cu at (34.0, 137.5)
- added kibuzzard-6AAFFF2E: G***, kibuzzard-6AAFFF2E, F.Cu at (33.9, 127.4)
- C42, C43: value 1u -> 10u; footprint Capacitor_SMD:C_0201_0603Metric -> Capacitor_SMD:C_1206_3216Metric
- C44: value 100n -> 10u; footprint Capacitor_SMD:C_0201_0603Metric -> Capacitor_SMD:C_1206_3216Metric
- R11: value 27K -> 27.4K
- R12: value 1M -> 2.49k
- R13: value 1M -> 280k
- SW2: value K8-5851S-N1 -> SW_Push; footprint lib:K8-5851S-N1 -> Button_Switch_SMD:SW_SPST_EVPBF
- U1: value TPS7A0533PDBV -> ICL7660; footprint Package_TO_SOT_SMD:SOT-23-5 -> Package_SO:SOIC-8_3.9x4.9mm_P1.27mm
- moved kibuzzard-6A01FB9A 65.1 mm to (103.0, 107.6)
- moved D1 58.1 mm to (103.0, 113.0), turned to -90 degrees
- moved SW2 56.6 mm to (103.0, 143.0), turned to 90 degrees
- moved C45 52.0 mm to (101.8, 117.2), turned to 180 degrees
- moved D2 44.0 mm to (103.0, 123.0), turned to -90 degrees
- moved C46 37.9 mm to (101.8, 127.2), turned to 180 degrees
- moved R12 36.6 mm to (86.6, 106.3), turned to 180 degrees
- moved C44 11.9 mm to (39.4, 119.6)
- moved U1 11.3 mm to (38.0, 115.4), turned to 0 degrees
- moved C48 10.9 mm to (32.2, 107.0), turned to 180 degrees
- moved R13 10.1 mm to (45.1, 106.3)
- moved A1 10.0 mm to (55.0, 93.0)
- moved C20 10.0 mm to (84.8, 120.5)
- moved C21 10.0 mm to (69.8, 120.5)
- moved C22 10.0 mm to (54.8, 120.5)
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Connections:
- A1 pad 35: Net-(A1-ADC_VREF) -> unconnected-(A1-ADC_VREF-Pad35)_1
- C43 pad 1: GND -> Net-(U1-CAP-)
- C43 pad 2: +3.3VADC -> Net-(U1-CAP+)
- C44 pad 2: +3.3VADC -> -VSYS
- D2 pad 4: Net-(D2-DOUT) -> unconnected-(D2-DOUT-Pad4)
- R12 pad 1: /ADC1 -> /COME
- SW2 pad 1: GND -> /~{START}
- SW2 pad 2: /~{START} -> GND
- U1 pad 1: VSYS -> unconnected-(U1-NC-Pad1)
- U1 pad 2: GND -> Net-(U1-CAP+)
- U1 pad 3: VSYS -> GND
- U1 pad 4: unconnected-(U1-NC-Pad4) -> Net-(U1-CAP-)
- U1 pad 5: +3.3VADC -> -VSYS
- U2 pad 16: GND -> -VSYS
- U3 pad 16: GND -> -VSYS
- U4 pad 16: GND -> -VSYS
Routing:
- net -VSYS: track 0.00 -> 61.2 mm, vias 0 -> 4
- net /LED_DIN: track 69.6 -> 115.0 mm, vias 0 -> 1
- net +3.3V: track 174.6 -> 217.5 mm, vias 4 -> 5
- net VSYS: track 284.2 -> 248.5 mm
- net Net-(A1-ADC_VREF): track 28.0 -> 0.00 mm
- net /~{START}: track 119.1 -> 100.7 mm, vias 0 -> 2
- net +3.3VADC: track 14.4 -> 0.00 mm
- net /COME: track 78.9 -> 90.6 mm
- net Net-(D2-DOUT): track 6.43 -> 0.00 mm
- net GND: track 42.4 -> 47.5 mm, vias 158 -> 139
- net /CON6: track 78.9 -> 82.3 mm
- net /COMC: track 69.4 -> 66.2 mm, vias 4 -> 5
- net Net-(U1-CAP+): track 0.00 -> 2.87 mm
- net Net-(U1-CAP-): track 0.00 -> 2.70 mm
- net /STB2: track 47.4 -> 45.1 mm
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Other:
- board size 80 x 100 mm -> 80 x 90 mm
