File: BondTest72.kicad_sch (KiCad schematic)
At the start: 39 parts, among them J1 Conn_01x07, J3 Conn_2Rows-41Pins_MountingPin, J4 Conn_2Rows-41Pins_MountingPin, SW1 SW_Push, SW2 K8-5851S-N1, SW3 K8-5851S-N1, U1 TPS7A0533PDBV, U2 CH446X, U3 CH446X, U4 CH446X

Commit message: - r2 update. Notes in README.md
Parts:
- removed C47: 100n, Capacitor_SMD:C_0201_0603Metric, symbol Device:C_Small
- removed D3: SK6812, LED_SMD:LED_SK6812_PLCC4_5.0x5.0mm_P3.2mm, symbol LED:SK6812
- removed JP3: SolderJumper_2_Open, Jumper:SolderJumper-2_P1.3mm_Open_TrianglePad1.0x1.5mm, symbol Jumper:SolderJumper_2_Open
- removed R10, R9: 1M, Resistor_SMD:R_0201_0603Metric, symbol Device:R_Small
- removed SW2, SW3: K8-5851S-N1, lib:K8-5851S-N1, symbol lib:SW_Push_DPDT_K8
- removed U1: TPS7A0533PDBV, Package_TO_SOT_SMD:SOT-23-5, symbol Regulator_Linear:TPS7A0533PDBV
- added C23, C24, C25: 100n, Capacitor_SMD:C_0201_0603Metric, symbol Device:C_Small
- added C50: 120pF, Capacitor_SMD:C_0201_0603Metric, symbol Device:C_Small
- added R14: 10k, Resistor_SMD:R_0201_0603Metric, symbol Device:R_Small
- added R15: 100k, Resistor_SMD:R_0201_0603Metric, symbol Device:R_Small
- added SW2: SW_Push, Button_Switch_SMD:SW_SPST_EVPBF, symbol Switch:SW_Push
- added U1: ICL7660, Package_SO:SOIC-8_3.9x4.9mm_P1.27mm, symbol Regulator_SwitchedCapacitor:ICL7660
- A1: Part Number Pico 2 -> C41407547
- C40, C41: Part Number C307385 -> C170153
- C42, C43: value 1u -> 10u; footprint Capacitor_SMD:C_0201_0603Metric -> Capacitor_SMD:C_1206_3216Metric; Part Number C307385 -> C9807
- C44: value 100n -> 10u; footprint Capacitor_SMD:C_0201_0603Metric -> Capacitor_SMD:C_1206_3216Metric; Part Number C76939 -> C9807
- J1: now not fitted
- J3, J4: Part Number C432807 -> C21261706
- R11: value 27K -> 27.4K; Part Number C273283 -> C273316
- R12: value 1M -> 2.49k; Part Number C4066408 -> C851701
- R13: value 1M -> 280k; Part Number C4066408 -> C778392
- U2, U3, U4: Part Number (none) -> C3018882
Connections:
- net +3.3V: now also R14.2
- net ADC1: now also C50.2; no longer R12.1
- net COME: now also R12.1
- net CON6: now also R15.2
- net GND: now also C23.1, C24.1, C25.1, C50.1, R15.1, SW2.2, U1.3 (GND); no longer C43.1, U2.16 (VEE), U3.16 (VEE), U4.16 (VEE)
- net VSYS: now also U1.8 (V+)
- net ~{START}: now also R14.1, SW2.1
- net +3.3VADC: no longer names the net of C43.2
- net +3.3VADC: now also U1.2 (CAP+); no longer C44.2
- new net: C43.1, U1.4 (CAP-)
- new net -VSYS: C23.2, C24.2, C25.2, C44.2, U1.5 (VOUT), U2.16 (VEE), U3.16 (VEE), U4.16 (VEE)
- no-connect marks 25 -> 28
Other:
- note added: "-VSYS regulator"
- note added: "2x RGB LED 1x push button"
- note added: "COMC - 10uA"
- note added: "COMD - 100uA current source"
- note added: "COME - 1000uA current source"
- note added: "Current is injected into the DUT GND pad 3 current sources, forward-biasing the VSS-side diode. The Bond Under Test (BuT) is grounded via COMB, completing the current path."
- note added: "Current sources & COMx mapping"
- note added: "Drive pico GPIO23 to improve ADC reference stability"
- note added: "PASS/FAIL"
- note added: "RP2350 A2 Errata"
- note added: "START"
- note removed: "1x red LED 1x yellow LED 1x green LED 1x push button 1x aux input"
- note removed: "COMC - Next bond (ADC2)"
- note removed: "COMD - Current source (ADC0)"
- note removed: "Current is injected into the DUT GND pad via COMD, forward-biasing the VSS-side diode. The Bond Under Test (BuT) is grounded via COMB, completing the current path. Neighbouring bonds (previous and next) are monitored to detect shorts to the BuT."
- note removed: "Current source & COMx mapping"
- note removed: "Drive GPIO23 to improve ADC reference stability"
- note removed: "External ADC reference"
- note removed: "FAIL"
- note removed: "PASS"
- note removed: "START (left)"
- note removed: "START (right)"
- moved on the sheet: C20, C21, C22, C48, NT1, NT2, NT3, R11, R13, U2, U3, U4
